File: ESP12E BMS.brd (EAGLE design)
At the start: 100 x 80 mm, 8 parts, among them Q1 IRFZ44N, X1 JST-XH-02-PIN-ROUND-PAD

Commit message: Add files via upload
Routing:
- net GND: track 66.1 -> 142.3 mm
- net 3V: track 0.00 -> 56.6 mm
Other:
- board size 100 x 80 mm -> 86.2 x 35.5 mm
Changed lines of the file:
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@@
 <board>
 <plain>
-<wire x1="0" y1="0" x2="100" y2="0" width="0" layer="20"/>
-<wire x1="100" y1="0" x2="100" y2="80" width="0" layer="20"/>
-<wire x1="100" y1="80" x2="0" y2="80" width="0" layer="20"/>
-<wire x1="0" y1="80" x2="0" y2="0" width="0" layer="20"/>
+<wire x1="13.97" y1="11.43" x2="100" y2="11.43" width="0" layer="20"/>
+<wire x1="100" y1="11.43" x2="100.127" y2="46.98" width="0" layer="20"/>
+<wire x1="100.127" y1="46.98" x2="14.097" y2="46.98" width="0" layer="20"/>
+<wire x1="14.097" y1="46.98" x2="13.97" y2="11.43" width="0" layer="20"/>
 </plain>
 <attributes>
@@
 <wire x1="63.5" y1="39.37" x2="67.31" y2="43.18" width="0.1524" layer="1"/>
 <wire x1="40.64" y1="39.37" x2="63.5" y2="39.37" width="0.1524" layer="1"/>
-<wire x1="67.31" y1="43.18" x2="85.09" y2="43.18" width="0" layer="19" extent="1-1"/>
-<wire x1="54.61" y1="15.24" x2="38.1" y2="27.94" width="0" layer="19" extent="1-1"/>
-<wire x1="74.93" y1="15.24" x2="54.61" y2="15.24" width="0" layer="19" extent="1-1"/>
-<wire x1="85.09" y1="15.24" x2="74.93" y2="15.24" width="0" layer="19" extent="1-1"/>
+<wire x1="38.1" y1="27.94" x2="41.91" y2="27.94" width="0.1524" layer="1"/>
+<wire x1="41.91" y1="27.94" x2="54.61" y2="15.24" width="0.1524" layer="1"/>
+<wire x1="54.61" y1="15.24" x2="57.15" y2="12.7" width="0.1524" layer="1"/>
+<wire x1="57.15" y1="12.7" x2="74.93" y2="12.7" width="0.1524" layer="1"/>
+<wire x1="74.93" y1="15.24" x2="74.93" y2="12.7" width="0.1524" layer="1"/>
+<wire x1="74.93" y1="12.7" x2="82.55" y2="12.7" width="0.1524" layer="1"/>
+<wire x1="82.55" y1="12.7" x2="85.09" y2="15.24" width="0.1524" layer="1"/>
+<wire x1="85.09" y1="43.18" x2="84.8968875" y2="43.18" width="0.1524" layer="1"/>
+<wire x1="67.5031125" y1="43.18" x2="67.31" y2="43.18" width="0.1524" layer="1"/>
+<wire x1="84.8968875" y1="43.18" x2="82.9918875" y2="41.275" width="0.1524" layer="1"/>
+<wire x1="69.4081125" y1="41.275" x2="67.5031125" y2="43.18" width="0.1524" layer="1"/>
+<wire x1="82.9918875" y1="41.275" x2="69.4081125" y2="41.275" width="0.1524" layer="1"/>
 </signal>
 <signal name="3V">
@@
 <contactref element="U$1" pad="16"/>
 <contactref element="U$1" pad="25"/>
-<wire x1="64.77" y1="43.18" x2="87.63" y2="43.18" width="0" layer="19" extent="1-1"/>
-<wire x1="77.47" y1="15.24" x2="87.63" y2="43.18" width="0" layer="19" extent="1-1"/>
+<wire x1="64.77" y1="43.18" x2="64.9631125" y2="43.18" width="0.1524" layer="1"/>
+<wire x1="87.4368875" y1="43.18" x2="87.63" y2="43.18" width="0.1524" layer="1"/>
+<wire x1="64.9631125" y1="43.18" x2="66.8681125" y2="45.085" width="0.1524" layer="1"/>
+<wire x1="85.5318875" y1="45.085" x2="87.4368875" y2="43.18" width="0.1524" layer="1"/>
+<wire x1="66.8681125" y1="45.085" x2="85.5318875" y2="45.085" width="0.1524" layer="1"/>
+<wire x1="87.63" y1="43.18" x2="87.63" y2="25.4" width="0.1524" layer="1"/>
+<wire x1="87.63" y1="25.4" x2="77.47" y2="15.24" width="0.1524" layer="1"/>
 </signal>
 <signal name="N$1">
