File: ESP12E BMS Low Voltage.brd (EAGLE design)
At the start: 96.2 x 35.5 mm, 9 parts, among them Q1 IRFZ44N, X1 JST-XH-02-PIN-ROUND-PAD

Commit message: Add files via upload
Parts:
- U$1: device nodemcu:NODEMCU -> nodemcuFix:NODEMCU
Connections:
- removed net +3V3: U$1.16, U$2.2
- removed net 3V: U$1.11, U$1.25
- new net 3V31: U$1.16
- new net 3V32: U$1.25
- new net GND1: U$1.10
- new net GND2: U$1.14
- new net GND3: U$1.17
- new net GND4: U$1.24
- new net N$7: U$1.11, U$2.2
- net GND: no longer U$1.10, U$1.14, U$1.17, U$1.24
Routing:
- net +3V3: track 107.9 -> 0.00 mm
- net GND: track 159.5 -> 65.5 mm
- net N$7: track 0.00 -> 72.5 mm
- net 3V: track 33.2 -> 0.00 mm
- net N$3: track 26.7 -> 21.5 mm
- net N$4: track 21.4 -> 20.6 mm
