File: ESP12E BMS Low Voltage.sch (EAGLE design)
At the start: 9 parts, among them Q1 IRFZ44N, X1 JST-XH-02-PIN-ROUND-PAD

Commit message: Add files via upload
Parts:
- U$1: device nodemcu:NODEMCU -> nodemcuFix:NODEMCU
Connections:
- removed net +3V3: U$1.3V@1, U$2.3.3V
- new net N$7: U$1.3V3, U$2.3V3
- net GND: now also U$1.GND; no longer U$1.GND@2
Other:
- moved on the sheet: X1-1, X1-2
Changed lines of the file:
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@@
 <parts>
 <part name="Q1" library="transistor-power" library_urn="urn:adsk.eagle:library:400" deviceset="PMOSFET_N" device="TO220BH" package3d_urn="urn:adsk.eagle:package:29490/1" value="IRFZ44N"/>
-<part name="U$1" library="nodemcu" deviceset="NODEMCU" device=""/>
+<part name="U$1" library="nodemcuFix" deviceset="NODEMCU" device=""/>
 <part name="X1" library="Rembrandt Electronics - JST XH Connectors v1-0" deviceset="JST-XH-02-PIN" device="-ROUND-PAD"/>
 <part name="LED1" library="led" library_urn="urn:adsk.eagle:library:259" deviceset="TLLR4400" device="" package3d_urn="urn:adsk.eagle:package:15797/1"/>
@@
 </instance>
 <instance part="U$1" gate="G$1" x="101.6" y="50.8" smashed="yes" rot="R90"/>
-<instance part="X1" gate="-2" x="58.42" y="30.48" smashed="yes">
-<attribute name="NAME" x="60.96" y="29.718" size="1.524" layer="95"/>
+<instance part="X1" gate="-2" x="58.42" y="35.56" smashed="yes">
+<attribute name="NAME" x="60.96" y="34.798" size="1.524" layer="95"/>
 </instance>
-<instance part="X1" gate="-1" x="58.42" y="33.02" smashed="yes">
-<attribute name="NAME" x="60.96" y="32.258" size="1.524" layer="95"/>
-<attribute name="VALUE" x="57.658" y="34.417" size="1.778" layer="96" display="off"/>
+<instance part="X1" gate="-1" x="58.42" y="38.1" smashed="yes">
+<attribute name="NAME" x="60.96" y="37.338" size="1.524" layer="95"/>
+<attribute name="VALUE" x="57.658" y="39.497" size="1.778" layer="96" display="off"/>
 </instance>
 <instance part="LED1" gate="G$1" x="50.8" y="68.58" smashed="yes">
@@
 </instance>
 <instance part="R1" gate="G$1" x="60.96" y="66.04" smashed="yes" rot="R270">
-<attribute name="NAME" x="62.4586" y="69.85" size="1.778" layer="95" rot="R270"/>
-<attribute name="VALUE" x="57.658" y="69.85" size="1.778" layer="96" rot="R270"/>
+<attribute name="NAME" x="57.3786" y="67.31" size="1.778" layer="95" rot="R270"/>
+<attribute name="VALUE" x="62.738" y="67.31" size="1.778" layer="96" rot="R270"/>
 </instance>
 <instance part="R2" gate="G$1" x="78.74" y="30.48" smashed="yes" rot="R180">
-<attribute name="NAME" x="82.55" y="28.9814" size="1.778" layer="95" rot="R180"/>
-<attribute name="VALUE" x="80.01" y="33.782" size="1.778" layer="96" rot="R180"/>
+<attribute name="NAME" x="80.01" y="28.9814" size="1.778" layer="95" rot="R180"/>
+<attribute name="VALUE" x="81.026" y="33.782" size="1.778" layer="96" rot="R180"/>
 </instance>
 <instance part="R3" gate="G$1" x="50.8" y="58.42" smashed="yes" rot="R90">
-<attribute name="NAME" x="49.3014" y="54.61" size="1.778" layer="95" rot="R90"/>
-<attribute name="VALUE" x="54.102" y="54.61" size="1.778" layer="96" rot="R90"/>
+<attribute name="NAME" x="49.3014" y="57.15" size="1.778" layer="95" rot="R90"/>
+<attribute name="VALUE" x="54.102" y="57.15" size="1.778" layer="96" rot="R90"/>
 </instance>
-<instance part="GND1" gate="1" x="116.84" y="27.94" smashed="yes">
-<attribute name="VALUE" x="114.3" y="25.4" size="1.778" layer="96"/>
+<instance part="GND1" gate="1" x="86.36" y="27.94" smashed="yes">
+<attribute name="VALUE" x="83.82" y="25.4" size="1.778" layer="96"/>
 </instance>
 <instance part="GND2" gate="1" x="58.42" y="53.34" smashed="yes">
@@
 <attribute name="VALUE" x="48.26" y="48.26" size="1.778" layer="96"/>
 </instance>
-<instance part="P+1" gate="1" x="33.02" y="53.34" smashed="yes">
-<attribute name="VALUE" x="33.02" y="53.34" size="1.778" layer="96" rot="R90"/>
+<instance part="P+1" gate="1" x="45.72" y="33.02" smashed="yes">
+<attribute name="VALUE" x="48.26" y="33.02" size="1.778" layer="96" rot="R90"/>
 </instance>
 <instance part="P+2" gate="1" x="78.74" y="58.42" smashed="yes">
@@
 </instance>
 <instance part="R4" gate="G$1" x="73.66" y="55.88" smashed="yes">
-<attribute name="NAME" x="69.85" y="57.3786" size="1.778" layer="95"/>
-<attribute name="VALUE" x="69.85" y="52.578" size="1.778" layer="96"/>
+<attribute name="NAME" x="72.39" y="57.3786" size="1.778" layer="95"/>
+<attribute name="VALUE" x="72.39" y="52.578" size="1.778" layer="96"/>
 </instance>
 <instance part="P+3" gate="1" x="73.66" y="33.02" smashed="yes">
 <attribute name="VALUE" x="73.66" y="33.02" size="1.778" layer="96" rot="R90"/>
 </instance>
-<instance part="P+4" gate="1" x="55.88" y="35.56" smashed="yes">
-<attribute name="VALUE" x="55.88" y="35.56" size="1.778" layer="96" rot="R90"/>
+<instance part="P+4" gate="1" x="55.88" y="40.64" smashed="yes">
+<attribute name="VALUE" x="55.88" y="40.64" size="1.778" layer="96" rot="R90"/>
 </instance>
-<instance part="GND4" gate="1" x="55.88" y="27.94" smashed="yes">
-<attribute name="VALUE" x="53.34" y="25.4" size="1.778" layer="96"/>
+<instance part="GND4" gate="1" x="55.88" y="33.02" smashed="yes">
+<attribute name="VALUE" x="53.34" y="30.48" size="1.778" layer="96"/>
 </instance>
-<instance part="U$2" gate="G$1" x="33.02" y="40.64" smashed="yes" rot="R180">
-<attribute name="VALUE" x="38.1" y="35.56" size="1.27" layer="94" rot="R180"/>
+<instance part="U$2" gate="G$1" x="40.64" y="43.18" smashed="yes">
+<attribute name="VALUE" x="35.56" y="48.26" size="1.27" layer="94"/>
 </instance>
-<instance part="GND5" gate="1" x="40.64" y="50.8" smashed="yes">
-<attribute name="VALUE" x="40.64" y="48.26" size="1.778" layer="96"/>
+<instance part="GND5" gate="1" x="33.02" y="27.94" smashed="yes">
+<attribute name="VALUE" x="30.48" y="25.4" size="1.778" layer="96"/>
 </instance>
 </instances>
@@
 </segment>
 <segment>
-<pinref part="U$1" gate="G$1" pin="GND@2"/>
-<pinref part="GND1" gate="1" pin="GND"/>
-</segment>
-<segment>
 <pinref part="X1" gate="-2" pin="S"/>
 <pinref part="GND4" gate="1" pin="GND"/>
 </segment>
 <segment>
+<pinref part="U$1" gate="G$1" pin="GND"/>
+<pinref part="GND1" gate="1" pin="GND"/>
+</segment>
+<segment>
 <pinref part="U$2" gate="G$1" pin="GND"/>
-<wire x1="38.1" y1="50.8" x2="38.1" y2="53.34" width="0.1524" layer="91"/>
 <pinref part="GND5" gate="1" pin="GND"/>
-<wire x1="38.1" y1="53.34" x2="40.64" y2="53.34" width="0.1524" layer="91"/>
+<wire x1="35.56" y1="33.02" x2="35.56" y2="30.48" width="0.1524" layer="91"/>
+<wire x1="35.56" y1="30.48" x2="33.02" y2="30.48" width="0.1524" layer="91"/>
 </segment>
 </net>
@@
 <segment>
 <pinref part="U$2" gate="G$1" pin="VIN"/>
+<wire x1="40.64" y1="33.02" x2="40.64" y2="30.48" width="0.1524" layer="91"/>
 <pinref part="P+1" gate="1" pin="V+"/>
+<wire x1="40.64" y1="30.48" x2="45.72" y2="30.48" width="0.1524" layer="91"/>
 </segment>
 </net>
@@
 <segment>
 <pinref part="R1" gate="G$1" pin="1"/>
-<wire x1="60.96" y1="71.12" x2="60.96" y2="76.2" width="0.1524" layer="91"/>
-<wire x1="60.96" y1="76.2" x2="86.36" y2="76.2" width="0.1524" layer="91"/>
+<wire x1="60.96" y1="71.12" x2="60.96" y2="73.66" width="0.1524" layer="91"/>
+<wire x1="60.96" y1="73.66" x2="86.36" y2="73.66" width="0.1524" layer="91"/>
 <pinref part="U$1" gate="G$1" pin="D1"/>
-<wire x1="86.36" y1="76.2" x2="86.36" y2="71.12" width="0.1524" layer="91"/>
+<wire x1="86.36" y1="73.66" x2="86.36" y2="71.12" width="0.1524" layer="91"/>
 </segment>
 </net>
@@
 <segment>
 <pinref part="LED1" gate="G$1" pin="A"/>
-<wire x1="50.8" y1="71.12" x2="50.8" y2="78.74" width="0.1524" layer="91"/>
+<wire x1="50.8" y1="71.12" x2="50.8" y2="76.2" width="0.1524" layer="91"/>
 <pinref part="U$1" gate="G$1" pin="D2"/>
-<wire x1="50.8" y1="78.74" x2="88.9" y2="78.74" width="0.1524" layer="91"/>
-<wire x1="88.9" y1="78.74" x2="88.9" y2="71.12" width="0.1524" layer="91"/>
+<wire x1="50.8" y1="76.2" x2="88.9" y2="76.2" width="0.1524" layer="91"/>
+<wire x1="88.9" y1="76.2" x2="88.9" y2="71.12" width="0.1524" layer="91"/>
 </segment>
 </net>
@@
 </segment>
 </net>
-<net name="+3V3" class="0">
+<net name="N$7" class="0">
 <segment>
-<pinref part="U$2" gate="G$1" pin="3.3V"/>
-<wire x1="35.56" y1="50.8" x2="35.56" y2="81.28" width="0.1524" layer="91"/>
-<pinref part="U$1" gate="G$1" pin="3V@1"/>
-<wire x1="35.56" y1="81.28" x2="119.38" y2="81.28" width="0.1524" layer="91"/>
-<wire x1="119.38" y1="81.28" x2="119.38" y2="71.12" width="0.1524" layer="91"/>
+<pinref part="U$2" gate="G$1" pin="3V3"/>
+<wire x1="38.1" y1="33.02" x2="38.1" y2="24.384" width="0.1524" layer="91"/>
+<wire x1="38.1" y1="24.384" x2="109.22" y2="24.384" width="0.1524" layer="91"/>
+<pinref part="U$1" gate="G$1" pin="3V3"/>
+<wire x1="109.22" y1="24.384" x2="109.22" y2="30.48" width="0.1524" layer="91"/>
 </segment>
 </net>
@@
 </sheet>
 </sheets>
+<errors>
+</errors>
 </schematic>
 </drawing>
